File: CAD/gba-zero.brd (EAGLE design)
At the start: 130.7 x 72.9 mm, 60 parts, among them J1 SWTCHCRFT_3.5JACK5-JACK-SMD, P1 50_PIN_CON, P3 LINK_CONNECTOR, Q1 BSS138, U1 APX803, U2 NC7WZ16, U3 74LVC2G02, U4 74LVC3G04, U5 LM4875, U6 RPI-ZEROSMD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

Commit message: add edited files by @Gameboypi :clap:
Parts:
- added S7: AB_BUTTON, gbz master:AB_BUTTON
Connections:
- new net BTN_X: S7.A@1, S7.A@2, U6.31
- new net BTN_Y: S7.B@1, S7.B@2, U6.35
- net GND: now also S7.GND@1, S7.GND@2, S7.GND@3, S7.GND@4
Routing:
- net BTN_X: track 0.00 -> 47.5 mm, vias 0 -> 1
- net BTN_Y: track 0.00 -> 42.0 mm, vias 0 -> 1
- net BTN_RS: track 50.3 -> 51.2 mm
Changed lines of the file:
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@@
 <?xml version="1.0" encoding="utf-8"?>
 <!DOCTYPE eagle SYSTEM "eagle.dtd">
-<eagle version="7.6.0">
+<eagle version="9.0.0">
 <drawing>
 <settings>
 <setting alwaysvectorfont="no"/>
+<setting keepoldvectorfont="yes"/>
 <setting verticaltext="up"/>
 </settings>
-<grid distance="0.01" unitdist="inch" unit="inch" style="lines" multiple="1" display="no" altdistance="0.001" altunitdist="inch" altunit="inch"/>
+<grid distance="0.01" unitdist="inch" unit="mil" style="lines" multiple="1" display="no" altdistance="0.001" altunitdist="mil" altunit="mil"/>
 <layers>
 <layer number="1" name="Top" color="4" fill="1" visible="yes" active="yes"/>
@@
 <layer number="59" name="tCarbon" color="7" fill="1" visible="yes" active="yes"/>
 <layer number="60" name="bCarbon" color="7" fill="1" visible="yes" active="yes"/>
+<layer number="88" name="SimResults" color="9" fill="1" visible="no" active="no"/>
+<layer number="89" name="SimProbes" color="9" fill="1" visible="no" active="no"/>
 <layer number="90" name="Modules" color="7" fill="1" visible="no" active="no"/>
 <layer number="91" name="Nets" color="2" fill="1" visible="no" active="no"/>
@@
 <layer number="154" name="FabDoc2" color="2" fill="1" visible="no" active="no"/>
 <layer number="155" name="FabDoc3" color="7" fill="15" visible="no" active="no"/>
+<layer number="166" name="AntennaArea" color="7" fill="1" visible="no" active="yes"/>
+<layer number="168" name="4mmHeightArea" color="7" fill="1" visible="no" active="yes"/>
 <layer number="191" name="mNets" color="7" fill="1" visible="yes" active="yes"/>
 <layer number="192" name="mBusses" color="7" fill="1" visible="yes" active="yes"/>
@@
 <hole x="19.422390625" y="18.10148125" drill="2.5"/>
 <hole x="13.641596875" y="27.388421875" drill="2.5"/>
-<hole x="120.9808375" y="37.2345625" drill="2.5"/>
-<hole x="115.854896875" y="47.952840625" drill="3.8"/>
 <circle x="113.0755" y="61.42" radius="2.6924" width="1.016" layer="51"/>
 <circle x="112.029784375" y="56.711425" radius="3.3528" width="0.0127" layer="22"/>
@@
 <classes>
 <class number="0" name="default" width="0" drill="0">
+</class>
+<class number="1" name="power" width="0.2794" drill="0">
 </class>
 </classes>
@@
 <param name="dpMaxLengthDifference" value="10mm"/>
 <param name="dpGapFactor" value="2.5"/>
-<param name="checkGrid" value="0"/>
 <param name="checkAngle" value="0"/>
 <param name="checkFont" value="1"/>
 <param name="checkRestrict" value="0"/>
+<param name="checkStop" value="0"/>
+<param name="checkValues" value="0"/>
 <param name="useDiameter" value="13"/>
 <param name="maxErrors" value="50"/>
@@
 <element name="C11" library="microbuilder" package="0603" value="10μF" x="38.1" y="39.37" rot="MR0"/>
 <element name="C14" library="microbuilder" package="0603" value="10μF" x="64.081659375" y="68.539359375" rot="MR0"/>
-<element name="U1" library="adafruit" package="SOT23" value="APX803" x="67.523359375" y="35.4076" smashed="yes" rot="R180">
+<element name="U1" library="adafruit" library_urn="urn:adsk.eagle:library:420" package="SOT23" value="APX803" x="67.523359375" y="35.4076" smashed="yes" rot="R180">
 <attribute name="NAME" x="71.206359375" y="36.0426" size="1.016" layer="25" font="vector" ratio="18" rot="R180"/>
 <attribute name="VALUE" x="65.618359375" y="36.6776" size="0.4064" layer="51" font="vector" ratio="10" rot="R180"/>
@@
 <element name="R12" library="microbuilder" package="0603" value="0" x="63.246" y="51.308" rot="R180"/>
 <element name="U$1" library="gba-zero-parts" package="SIGNATURE" value="SIGNATURE" x="124.4854" y="44.831" rot="MR0"/>
+<element name="S7" library="gbz master" package="AB_BUTTON" value="AB_BUTTON" x="119.531615625" y="42.061690625" rot="R91.2"/>
 </elements>
 <signals>
@@
 <contactref element="C2" pad="2"/>
 <contactref element="C4" pad="2"/>
+<contactref element="S7" pad="GND@3"/>
+<contactref element="S7" pad="GND@4"/>
+<contactref element="S7" pad="GND@1"/>
+<contactref element="S7" pad="GND@2"/>
 </signal>
 <signal name="MISO">
@@
 <wire x1="88.646" y1="42.1005" x2="88.646" y2="45.2882" width="0.254" layer="16"/>
 <via x="88.646" y="45.2882" extent="1-16" drill="0.6" shape="square"/>
-<wire x1="88.646" y1="45.2882" x2="118.4402" y2="45.2882" width="0.254" layer="1"/>
-<wire x1="126.149890625" y1="58.077890625" x2="125.476" y2="57.404" width="0.254" layer="1"/>
-<wire x1="125.476" y1="57.404" x2="125.476" y2="52.324" width="0.254" layer="1"/>
-<wire x1="125.476" y1="52.324" x2="118.4402" y2="45.2882" width="0.254" layer="1"/>
+<wire x1="125.476" y1="57.404" x2="126.149890625" y2="58.077890625" width="0.254" layer="1"/>
 <wire x1="126.149890625" y1="58.077890625" x2="126.149890625" y2="59.274340625" width="0.254" layer="1"/>
 <wire x1="126.149890625" y1="59.274340625" x2="126.200178125" y2="59.324628125" width="0.254" layer="1"/>
+<wire x1="88.646" y1="45.2882" x2="119.9642" y2="45.2882" width="0.254" layer="1"/>
+<wire x1="119.9642" y1="45.2882" x2="125.476" y2="50.8" width="0.254" layer="1"/>
+<wire x1="125.476" y1="50.8" x2="125.476" y2="57.404" width="0.254" layer="1"/>
 </signal>
 <signal name="BTN_L">
@@
 <wire x1="61.8938" y1="50.8058" x2="62.396" y2="51.308" width="0.254" layer="1"/>
 </signal>
+<signal name="BTN_X">
+<contactref element="S7" pad="A@2"/>
+<contactref element="S7" pad="A@1"/>
+<contactref element="U6" pad="31"/>
+<via x="83.058" y="49.454" extent="1-16" drill="0.6" shape="square"/>
+<wire x1="80.9752" y1="42.1005" x2="80.9752" y2="47.3712" width="0.254" layer="16"/>
+<wire x1="80.9752" y1="47.3712" x2="83.058" y2="49.454" width="0.254" layer="16"/>
+<wire x1="83.058" y1="49.454" x2="86.182" y2="52.578" width="0.254" layer="1"/>
+<wire x1="86.182" y1="52.578" x2="104.902" y2="52.578" width="0.254" layer="1"/>
+<wire x1="108.094559375" y1="49.385440625" x2="114.781765625" y2="49.385440625" width="0.254" layer="1"/>
+<wire x1="104.902" y1="52.578" x2="108.094559375" y2="49.385440625" width="0.254" layer="1"/>
+<wire x1="117.146825" y1="46.19449375" x2="115.85750625" y2="46.19449375" width="0.254" layer="1"/>
+<wire x1="115.85750625" y1="46.19449375" x2="114.808" y2="47.244" width="0.254" layer="1"/>
+<wire x1="114.808" y1="47.244" x2="114.808" y2="49.35920625" width="0.254" layer="1"/>
+<wire x1="114.808" y1="49.35920625" x2="114.781765625" y2="49.385440625" width="0.254" layer="1"/>
+</signal>
+<signal name="BTN_Y">
+<contactref element="S7" pad="B@2"/>
+<contactref element="S7" pad="B@1"/>
+<contactref element="U6" pad="35"/>
+<wire x1="119.38" y1="36.385175" x2="119.535609375" y2="36.385175" width="0.254" layer="1"/>
+<wire x1="86.106" y1="41.91" x2="86.106" y2="41.402" width="0.254" layer="1"/>
+<via x="86.106" y="42.164" extent="1-16" drill="0.6" shape="square"/>
+<wire x1="86.106" y1="41.402" x2="91.6638" y2="35.8442" width="0.254" layer="1"/>
+<wire x1="118.839025" y1="35.8442" x2="119.38" y2="36.385175" width="0.254" layer="1"/>
+<wire x1="91.6638" y1="35.8442" x2="118.839025" y2="35.8442" width="0.254" layer="1"/>
+<wire x1="121.743446875" y1="33.35145" x2="121.90066875" y2="33.194228125" width="0.254" layer="1"/>
+<wire x1="119.38" y1="34.036" x2="120.06455" y2="33.35145" width="0.254" layer="1"/>
+<wire x1="120.06455" y1="33.35145" x2="121.743446875" y2="33.35145" width="0.254" layer="1"/>
+<wire x1="119.38" y1="36.385175" x2="119.38" y2="34.036" width="0.254" layer="1"/>
+<wire x1="86.106" y1="42.164" x2="86.106" y2="41.91" width="0.1524" layer="1"/>
+<wire x1="86.0552" y1="42.1005" x2="86.0552" y2="42.1132" width="0.1524" layer="16"/>
+<wire x1="86.0552" y1="42.1132" x2="86.106" y2="42.164" width="0.1524" layer="16"/>
+</signal>
 </signals>
-<errors>
-</errors>
 </board>
 </drawing>
@@
 which will not be processed correctly with this version.
 </note>
+<note version="8.2" severity="warning">
+Since Version 8.2, EAGLE supports online libraries. The ids
+of those online libraries will not be understood (or retained)
+with this version.
+</note>
 </compatibility>
