File: CAD/gba-zero.sch (EAGLE design)
At the start: 60 parts, among them J1 SWTCHCRFT_3.5JACK5-JACK-SMD, P1 50_PIN_CON, P3 LINK_CONNECTOR, Q1 BSS138, U1 APX803, U2 NC7WZ16, U3 74LVC2G02, U4 74LVC3G04, U5 LM4875, U6 RPI-ZEROSMD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

Commit message: add edited files by @Gameboypi :clap:
Parts:
- added S7: AB_BUTTON, gbz master:AB_BUTTON
Connections:
- new net BTN_X: S7.A, U6.GPIO6
- new net BTN_Y: S7.B, U6.GPIO19
- net GND: now also S7.GND
